File: card-extender/card-extender.kicad_pcb (KiCad board)
At the start: 2 copper layers, 240 x 227 mm, 15 parts, among them J1 Card_Edge_1x44, J2 Card_Edge_1x44, J3 Conn_01x22_Pin, J4 Conn_01x22_Pin, J5 Card_Edge_1x44, J6 Card_Edge_1x44, J7 Conn_01x22_Pin, J8 Conn_01x22_Pin

Commit message: adding 3d model for socket connector
Parts:
- J6: footprint Korg PS-3x00 KLM Cards:CardEdge-2x22_2.18x9.75mm_P3.96mm -> Korg PS-3x00 KLM Cards:CardSocket-2x22_P3.96mm
Changed lines of the file:
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@@
 		)
 	)
-	(footprint "Korg PS-3x00 KLM Cards:CardEdge-2x22_2.18x9.75mm_P3.96mm"
+	(footprint "Korg PS-3x00 KLM Cards:CardSocket-2x22_P3.96mm"
 		(layer "F.Cu")
 		(at 200 25 90)
-		(descr "CardEdge-2x22: 2.18mm plated traces on PCB for card-edge; 44 leads; body width 2x89mm w 31mm gap")
-		(tags "CardEdge 2x22 3.96mm")
+		(descr "CardSocket-2x22: 44 pins; 3.96mm pitch")
+		(tags "CardSocket 2x22 44 pins; 3.96mm pitch")
 		(property "Reference" "J6"
-			(at 4.191 0 0)
+			(at 4.191 0 180)
 			(layer "B.SilkS")
 			(effects
@@
 		)
 		(property "Value" "Card_Edge_1x44"
-			(at -3.937 0 0)
+			(at -3.937 0 180)
 			(layer "B.Fab")
 			(effects
@@
 			)
 		)
-		(property "Footprint" "Korg PS-3x00 KLM Cards:CardEdge-2x22_2.18x9.75mm_P3.96mm"
+		(property "Footprint" "Korg PS-3x00 KLM Cards:CardSocket-2x22_P3.96mm"
 			(at 0 0 90)
 			(unlocked yes)
@@
 		)
 		(fp_text user "${REFERENCE}"
-			(at 0 0 0)
+			(at 0 0 180)
 			(layer "B.Fab")
 			(effects
@@
 			(pintype "passive")
 		)
+		(model "/home/dkaiser/code/pscards/klib/footprints/_ _M22DREH.STEP"
+			(offset
+				(xyz 11 114.5 -5)
+			)
+			(scale
+				(xyz 1 1 1)
+			)
+			(rotate
+				(xyz 0 0 90)
+			)
+		)
+		(model "/home/dkaiser/code/pscards/klib/footprints/_ _M22DREH.STEP"
+			(offset
+				(xyz 11 -6 -5)
+			)
+			(scale
+				(xyz 1 1 1)
+			)
+			(rotate
+				(xyz 0 0 90)
+			)
+		)
 	)
