File: card-extender/extender-side.kicad_sch (KiCad schematic)
At the start: 4 parts, among them J1 Card_Edge_1x44, J2 Card_Edge_1x44, J3 Conn_01x22_Pin, J4 Conn_01x22_Pin

Commit message: adding attribution fields
Other:
- company: (none) -> David Kaiser <dkaiser@dkaiser.org>
- title: (none) -> Korg PS Synth Card Extender
Changed lines of the file:
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@@
 	(generator_version "8.0")
 	(paper "A4")
+	(title_block
+		(title "Korg PS Synth Card Extender")
+		(date "2024-07-23")
+		(rev "1")
+		(company "David Kaiser <dkaiser@dkaiser.org>")
+		(comment 1 "Created with 'Korg PS-3x00 KLM Cards' template: https://github.com/ddkaiser/pscards")
+	)
 	(wire
 		(pts
